File: ThrottleAdapterBoard/ThrottleAdapterBoard.kicad_pcb (KiCad board)
At the start: 2 copper layers, 156.3 x 56.1 mm, 18 parts, among them J1 LCD5110, J2 POWER, J3 WemosS2MiniA, J4 WemosS2MiniB, J5 WemosS2MiniC, J6 WemosS2MiniD, J7 Keypad, J8 BAT_HOLDER, SW1 SW_SPDT

Commit message: PCB Board
Parts:
- added C1: 100nF, Capacitor_SMD:C_1210_3225Metric_Pad1.33x2.70mm_HandSolder, F.Cu at (129.1, 80.7)
- added C2: 100nF, Capacitor_SMD:C_1210_3225Metric_Pad1.33x2.70mm_HandSolder, F.Cu at (129.2, 94.0)
- added Q1: BC547, Package_TO_SOT_THT:TO-92_Inline_Horizontal1, B.Cu at (118.5, 85.3)
- added R2: 1k, Resistor_SMD:R_1206_3216Metric_Pad1.30x1.75mm_HandSolder, F.Cu at (113.7, 92.0)
- added R3: 10k, Resistor_SMD:R_1206_3216Metric_Pad1.30x1.75mm_HandSolder, F.Cu at (113.7, 88.4)
- added R4: 10k, Resistor_SMD:R_1206_3216Metric_Pad1.30x1.75mm_HandSolder, F.Cu at (124.9, 94.1)
- added R5: 10k, Resistor_SMD:R_1206_3216Metric_Pad1.30x1.75mm_HandSolder, F.Cu at (124.8, 80.9)
- added SW2: KY-040, Rotary_Encoder:RotaryEncoder_Alps_EC12E-Switch_Vertical_H20mm_CircularMountingHoles, F.Cu at (133.5, 84.8)
- J8: moved to B.Cu
- R1: value 600R -> 1k
- SW1: value SW_SPDT -> JS102011SAQN
- moved F1 28.3 mm to (125.6, 105.4)
- moved R1 9.64 mm to (113.7, 84.5), turned to 180 degrees
- moved J2 1.13 mm to (116.6, 96.7)
Connections:
- J3 pad 1: unconnected-(J3-Pin_1-Pad1) -> ENC_A
- J3 pad 2: unconnected-(J3-Pin_2-Pad2) -> ENC_B
- J3 pad 3: unconnected-(J3-Pin_3-Pad3) -> ENC_SW
- J4 pad 1: unconnected-(J4-Pin_1-Pad1) -> BLON
Routing:
- net ENC_SW: track 0.00 -> 77.8 mm, vias 0 -> 1
- net ENC_A: track 0.00 -> 73.6 mm
- net ENC_B: track 0.00 -> 55.2 mm
- net +BATT: track 9.00 -> 40.8 mm
- net Net-(SW1-B): track 43.5 -> 13.0 mm
- net BLON: track 0.00 -> 23.2 mm, vias 0 -> 1
- net +3.3V: track 75.3 -> 98.0 mm, vias 1 -> 2
- net BL: track 44.3 -> 28.2 mm
- net VCC: track 25.1 -> 33.1 mm, vias 1 -> 0
- net Net-(Q1-B): track 0.00 -> 7.66 mm
- net ROW2: track 136.5 -> 142.6 mm
- net ROW4: track 148.2 -> 143.1 mm
- net ROW3: track 138.6 -> 143.4 mm
- net COL1: track 143.9 -> 139.9 mm
- net COL3: track 144.0 -> 145.4 mm
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Other:
- outline, holes or cut-outs redrawn
- board text added: "Z21 Throttle Adapter made by stefan/strofo @2026 v1.1"
- board text removed: "Z21 Throttle Adapter ESP32 S3 Mini @2026 v1.0"
