File: ThrottleAdapterBoard/ThrottleAdapterBoard.kicad_sch (KiCad schematic)
At the start: 18 parts, among them J1 LCD5110, J2 POWER, J3 WemosS2MiniA, J4 WemosS2MiniB, J5 WemosS2MiniC, J6 WemosS2MiniD, J7 Keypad, J8 BAT_HOLDER, SW1 SW_SPDT

Commit message: PCB Board
Parts:
- added C1, C2: 100nF, Capacitor_SMD:C_1210_3225Metric_Pad1.33x2.70mm_HandSolder, symbol Device:C_Small
- added Q1: BC547, Package_TO_SOT_THT:TO-92_Inline_Horizontal1, symbol Transistor_BJT:BC547
- added R2: 1k, Resistor_SMD:R_1206_3216Metric_Pad1.30x1.75mm_HandSolder, symbol Device:R_Small
- added R3, R4, R5: 10k, Resistor_SMD:R_1206_3216Metric_Pad1.30x1.75mm_HandSolder, symbol Device:R_Small
- added SW2: KY-040, Rotary_Encoder:RotaryEncoder_Alps_EC12E-Switch_Vertical_H20mm_CircularMountingHoles, symbol Device:RotaryEncoder_Switch_MP
- R1: value 600R -> 1k
- SW1: value SW_SPDT -> JS102011SAQN
Connections:
- net +3.3V: now also Q1.1 (C), R4.1, R5.2
- net GND: now also C1.2, C2.2, Q1.3 (E), R3.2, SW2.C, SW2.MP, SW2.S2
- net BLON: now reaches J4.1 (Pin_1)
- net BLON: now also R2.2
- net ENC_A: now reaches J3.1 (Pin_1)
- net ENC_A: now also C1.1, R5.1, SW2.A
- net ENC_B: now reaches J3.2 (Pin_2)
- net ENC_B: now also C2.1, R4.2, SW2.B
- net ENC_SW: now reaches J3.3 (Pin_3)
- net ENC_SW: now also SW2.S1
- new net: Q1.2 (B), R2.1, R3.1
Other:
- note added: "POT USED FOR SPEED"
- moved on the sheet: R1
